Commit message: use a revolute joint to set the pitch

File: acq4/devices/geometries/sensapex_lefthanded.urdf (robot description, URDF)
Before this commit: robot sensapex_manipulator, 5 links, 4 joints
Links:
- added link xz_rotation_link; visual box size=0.005 0.005 0.005
Joints:
- added joint xz_rotation: type revolute, parent z_axis_link, child xz_rotation_link, axis 0 1 0, limit lower=-1.57 upper=1.57 effort=1000 velocity=0.5
- joint x_axis_joint: parent z_axis_link -> xz_rotation_link
